Commit message: urdf_for_auto_collision

File: description_files/urdf/g1_29dof.urdf (robot description, URDF)
Before this commit: robot g1_29dof_rev_1_0, 57 links, 56 joints
Links:
- link left_elbow_link: geometry collision cylinder length=0.13 radius=0.035; visual mesh filename=package://g1pilot/description_files/meshes/left_elbow_link.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
- link left_hip_pitch_link: geometry collision cylinder length=0.08 radius=0.04; visual mesh filename=package://g1pilot/description_files/meshes/left_hip_pitch_l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
- link left_hip_roll_link: geometry collision cylinder length=0.12 radius=0.07; visual mesh filename=package://g1pilot/description_files/meshes/left_hip_roll_li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
- link left_hip_yaw_link: geometry collision cylinder length=0.18 radius=0.055; visual mesh filename=package://g1pilot/description_files/meshes/left_hip_yaw_lin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
- link left_knee_link: geometry collision cylinder length=0.30 radius=0.06; visual mesh filename=package://g1pilot/description_files/meshes/left_knee_link.S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
- link left_rubber_hand: geometry collision box size=0.15 0.08 0.12; visual mesh filename=package://g1pilot/description_files/meshes/left_rubber_hand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
- link left_shoulder_yaw_link: geometry collision cylinder length=0.145 radius=0.04; visual mesh filename=package://g1pilot/description_files/meshes/left_shoulder_ya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
- link left_wrist_pitch_link: geometry collision cylinder length=0.10 radius=0.03; visual mesh filename=package://g1pilot/description_files/meshes/left_wrist_pitch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
- link left_wrist_roll_link: geometry collision cylinder length=0.056 radius=0.03; visual mesh filename=package://g1pilot/description_files/meshes/left_wrist_roll_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
- link left_wrist_yaw_link: geometry collision cylinder length=0.06 radius=0.03; visual mesh filename=package://g1pilot/description_files/meshes/left_wrist_yaw_l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
- link pelvis_contour_link: geometry collision box size=0.12 0.14 0.12; visual mesh filename=package://g1pilot/description_files/meshes/pelvis_contour_l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
- link right_elbow_link: geometry collision cylinder length=0.13 radius=0.035; visual mesh filename=package://g1pilot/description_files/meshes/right_elbow_link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
- link right_hip_pitch_link: geometry collision cylinder length=0.08 radius=0.04; visual mesh filename=package://g1pilot/description_files/meshes/right_hip_pitch_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
- link right_hip_roll_link: geometry collision cylinder length=0.12 radius=0.07; visual mesh filename=package://g1pilot/description_files/meshes/right_hip_roll_l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
- link right_hip_yaw_link: geometry collision cylinder length=0.18 radius=0.055; visual mesh filename=package://g1pilot/description_files/meshes/right_hip_yaw_li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
- link right_knee_link: geometry collision cylinder length=0.30 radius=0.06; visual mesh filename=package://g1pilot/description_files/meshes/right_knee_link.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
- link right_rubber_hand: geometry collision box size=0.15 0.08 0.12; visual mesh filename=package://g1pilot/description_files/meshes/right_rubber_han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
- link right_shoulder_yaw_link: geometry collision cylinder length=0.145 radius=0.04; visual mesh filename=package://g1pilot/description_files/meshes/right_shoulder_y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
- link right_wrist_pitch_link: geometry collision cylinder length=0.10 radius=0.03; visual mesh filename=package://g1pilot/description_files/meshes/right_wrist_pitc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
- link right_wrist_roll_link: geometry collision cylinder length=0.056 radius=0.03; visual mesh filename=package://g1pilot/description_files/meshes/right_wrist_roll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
- link right_wrist_yaw_link: geometry collision cylinder length=0.06 radius=0.03; visual mesh filename=package://g1pilot/description_files/meshes/right_wrist_yaw_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
- link torso_link: geometry collision box size=0.13 0.20 0.30; visual mesh filename=package://g1pilot/description_files/meshes/torso_link_rev_1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
- link waist_roll_link: geometry collision cylinder length=0.024 radius=0.017; visual mesh filename=package://g1pilot/description_files/meshes/waist_roll_link_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
- link waist_yaw_link: geometry collision cylinder length=0.15 radius=0.06; visual mesh filename=package://g1pilot/description_files/meshes/waist_yaw_link_r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
